File: Gerber/2ButtonKeyboardPCB.kicad_pcb (KiCad board)
At the start: 2 copper layers, 47.6 x 61.1 mm, 20 parts, among them SW1 SW_Push, U1 ATmega32U4-AU, Y1 16MHz

Commit message: Pcb Routing Update
Parts:
- moved SW1 39.2 mm to (155.6, 102.4), turned to 180 degrees
- moved F1 15.0 mm to (150.8, 89.7), turned to 90 degrees
- moved R1 3.99 mm to (160.2, 52.4)
- moved R4 3.70 mm to (167.5, 106.4), turned to 0 degrees
- moved R2 3.37 mm to (160.2, 55.6)
- moved C2 3.14 mm to (174.1, 87.5), turned to 0 degrees
Routing:
- net Net-(R3-Pad2): track 13.8 -> 37.5 mm, vias 0 -> 2
- net +5V: track 98.5 -> 117.8 mm, vias 4 -> 8
- net Net-(R2-Pad1): track 59.8 -> 49.0 mm
- net VCC: track 63.5 -> 55.0 mm
- net Net-(R1-Pad1): track 60.8 -> 52.3 mm
- net GND: track 174.4 -> 181.9 mm, vias 0 -> 1
- net D-: track 10.4 -> 13.4 mm
- net COL1: track 53.5 -> 51.1 mm
- net D+: track 11.6 -> 13.9 mm
- net Net-(R4-Pad2): track 3.14 -> 5.40 mm
- net COL0: track 44.6 -> 43.6 mm
